File: assets/pcbs/actuators-rev1/actuators-rev1.sch (KiCad schematic (older format))
At the start: 14 parts, among them J2 Screw_Terminal_01x02, J3 Screw_Terminal_01x02, J5 40HAT, J6 Conn_01x02, J7 Screw_Terminal_01x02, U1 ULN2003A, U2 PDQ15-Q24-S5-D

Commit message: Added v1 of pcbs and revision history readme
Parts:
- removed C1: CP1, Capacitor_THT:CP_Radial_D5.0mm_P2.00mm, symbol Device:CP1
- removed C2, C3: CP1, Capacitor_THT:CP_Radial_D5.0mm_P2.50mm, symbol Device:CP1
- added J1: Screw_Terminal_01x02, TerminalBlock:TerminalBlock_Altech_AK300-2_P5.00mm, symbol Connector:Screw_Terminal_01x02
- added J10, J4, J8, J9: Conn_01x02, Connector_PinHeader_2.54mm:PinHeader_1x02_P2.54mm_Vertical, symbol Connector_Generic:Conn_01x02
Connections:
- net labels added: +3.3V
- wire segments 84 -> 89
- no-connect marks 28 -> 0
Other:
- moved on the sheet: J6
