File: assets/pcbs/actuators-rev2/actuators-rev2.kicad_pcb (KiCad board)
At the start: 4 copper layers, 65 x 56 mm, 14 parts, among them J2 Screw_Terminal_01x02, J3 Screw_Terminal_01x02, J5 40HAT, J6 Conn_01x02, J7 Screw_Terminal_01x02, U1 ULN2003A, U2 PDQ15-Q24-S5-D

Commit message: Added v1 of pcbs and revision history readme
Other:
- net class Default removed
- board text added: "Tiger Vents Actuator Board Rev 2.0"
- board text removed: "Tiger Vents Actuator Board Rev 1.0"
